File: pcb/v0.1/purple-owl.kicad_pcb (KiCad board)
At the start: 2 copper layers, 291.4 x 94.3 mm, 124 parts, among them SW1 SW_Push, SW10 SW_Push, SW11 SW_Push, SW12 SW_Push, SW13 SW_Push, SW14 SW_Push, SW15 SW_Push, SW16 SW_Push, SW17 SW_Push, SW18 SW_Push, SW19 SW_Push, SW2 SW_Push, SW20 SW_Push, SW21 SW_Push, SW22 SW_Push, SW23 SW_Push, SW24 SW_Push, SW25 SW_Push, SW26 SW_Push, SW27 SW_Push, SW28 SW_Push, SW29 SW_Push, SW3 SW_Push, SW30 SW_Push, SW31 SW_Push, SW32 SW_Push, SW33 SW_Push, SW34 SW_Push, SW35 SW_Push, SW36 SW_Push, SW37 SW_Push, SW38 SW_Push, SW39 SW_Push, SW4 SW_Push, SW40 SW_Push, SW41 SW_Push, SW42 SW_Push, SW43 SW_Push, SW44 SW_Push, SW45 SW_Push, SW46 SW_Push, SW47 SW_Push, SW48 SW_Push, SW49 SW_Push, SW5 SW_Push, SW50 SW_Push, SW51 SW_Push, SW52 SW_Push, SW53 SW_Push, SW54 SW_Push, SW55 SW_Push, SW56 SW_Push, SW57 SW_Push, SW58 SW_Push, SW59 SW_Push, SW6 SW_Push, SW60 SW_Push, SW61 SW_Push, SW7 SW_Push, SW8 SW_Push, SW9 SW_Push, U1 Waveshare_RP2040_Zero

Commit message: Open pcb design for v1.0
- Schematic for v1.0 with 74HC165 shift registers for the 61 keys
- Matrix is polled using 5 pins - 3V3, GND, Latch, Data and Clock
- Solder jumper for 3V3 compatibility between KB2040 (ProMicro variant)
and QTPy layout (Waveshare RP2040 Zero, Pimoroni Tiny RP2040, Seeed Xiao
RP2040)
- Alternate few-pin footprints for Adafruit QTPy RP2040 and KB2040
 marking only pins required (functional and mechanical) for v1.0
- Smaller drill holes for the Alt footprints - 0.7/1.4mm
Other:
- board text added: "This is a prototype of the Purple Owl layout powered by a Waveshare RP2040 Zero. Eventually, the active electronics will go on the keyboard PCB itself. The uC board is tilted 26' which is approximately the slant of the columns. The 90' arcs softening the corners are 50mil radius."
- board text removed: "This is a prototype of the Purple Owl layout powered by a Waveshare RP2040 Zero. Eventually, the active electronins will go on the keyboard PCB itself. The uC board is tilted 26' which is approximately the slant of the columns. The 90' arcs softening the corners are 50mil radius."
Changed lines of the file:
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@@
     (effects (font (size 1.5 1.5) (thickness 0.3)))
   )
-  (gr_text "This is a prototype of the Purple Owl layout powered by a Waveshare RP2040 Zero.\nEventually, the active electronins will go on the keyboard PCB itself.\n\nThe uC board is tilted 26' which is approximately the slant of the columns.\n\nThe 90' arcs softening the corners are 50mil radius." (at 302.895 213.995) (layer "Dwgs.User")
+  (gr_text "This is a prototype of the Purple Owl layout powered by a Waveshare RP2040 Zero.\nEventually, the active electronics will go on the keyboard PCB itself.\n\nThe uC board is tilted 26' which is approximately the slant of the columns.\n\nThe 90' arcs softening the corners are 50mil radius." (at 302.895 213.995) (layer "Dwgs.User")
     (effects (font (size 1.5 1.5) (thickness 0.15)) (justify left))
   )
